File: pcb/controller/src/OWL - Rotor v2.kicad_pcb (KiCad board)
At the start: 4 copper layers, 60 x 60 mm, 118 parts, among them IC1 USB2422-I_MJ, J1 Motor, J3 USB_C_Receptacle_USB2.0_14P, J4 Slip Ring, J5 781715006, J6 SM03B-SRSS-TB, J8 Micro_SD_Card, J9 SM04B-SRSS-TB_LF__SN_, SW1 BOOTSEL, SW2 RESET, SW3 USER, U1 AP2112K-3.3, U2 LM66200DRLR, U3 PDRV8311HRRWR, U4 RP2354B, U5 USBLC6-2P6, U6 <value>, Y1 ABM8-272-T3, Y2 7M-24.000MAAJ-T

Commit message: Add manufacturer, MPN and LCSC part numbers to all boards
Part numbers taken from the matched JLCPCB order BOMs. Also mark the RM2
module (U6) and microSD socket (J8) as DNP, exclude test points from the
BOM, use KT-0805B for D7, 100n 50V for C42 as built, and set ENIG as the
surface finish.

Co-Authored-By: Claude Opus 5 <noreply@anthropic.com>
Parts:
- C42: value 100n 250V -> 100n 50V
- D7: value XL-1608UBC-04 -> KT-0805B
