File: pcb/controller/src/OWL - Rotor v2.kicad_pcb (KiCad board)
At the start: 4 copper layers, 60 x 60 mm, 118 parts, among them IC1 USB2422-I_MJ, J1 Motor, J3 USB_C_Receptacle_USB2.0_14P, J4 Slip Ring, J5 781715006, J6 SM03B-SRSS-TB, J8 Micro_SD_Card, J9 SM04B-SRSS-TB_LF__SN_, SW1 BOOTSEL, SW2 RESET, SW3 USER, U1 AP2112K-3.3, U2 LM66200DRLR, U3 PDRV8311HRRWR, U4 RP2354B, U5 USBLC6-2P6, U6 <value>, Y1 ABM8-272-T3, Y2 7M-24.000MAAJ-T

Commit message: Lower the current of the green 5V and 3.3V LEDs
R3 510 -> 1.43k and R40 150 -> 360, about 1.5 mA like the VM LED
instead of 3-4 mA. Both values are already in the BOM.

Co-Authored-By: Claude Opus 5 <noreply@anthropic.com>
Parts:
- R3: value 510 -> 1.43k
- R40: value 150 -> 360
Changed lines of the file:
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@@
 			)
 		)
-		(property "Value" "150"
+		(property "Value" "360"
 			(at 0 1.17 0)
 			(layer "F.Fab")
@@
 			)
 		)
-		(property "Manufacturer" "UNI-ROYAL"
+		(property "Manufacturer" "FOJAN"
 			(at 0 0 0)
 			(unlocked yes)
@@
 			)
 		)
-		(property "MPN" "0402WGF1500TCE"
+		(property "MPN" "FRC0402F3600TS"
 			(at 0 0 0)
 			(unlocked yes)
@@
 			)
 		)
-		(property "LCSC" "C25082"
+		(property "LCSC" "C2930003"
 			(at 0 0 0)
 			(unlocked yes)
@@
 			)
 		)
-		(property "Value" "510"
+		(property "Value" "1.43k"
 			(at 0 1.17 45)
 			(layer "F.Fab")
@@
 			)
 		)
-		(property "Manufacturer" "UNI-ROYAL"
+		(property "Manufacturer" "Yageo"
 			(at 0 0 0)
 			(unlocked yes)
@@
 			)
 		)
-		(property "MPN" "0402WGF5100TCE"
+		(property "MPN" "RC0402FR-071K43L"
 			(at 0 0 0)
 			(unlocked yes)
@@
 			)
 		)
-		(property "LCSC" "C25123"
+		(property "LCSC" "C163483"
 			(at 0 0 0)
 			(unlocked yes)

Commit message: Ship the controller VBUS jumper JP1 open
With both USB VBUS and the regulator connected, the LM66200 keeps
switching between the two nearly equal inputs and the 5V rail gets
noisy. JP1 is now an open solder jumper, so the controller runs from
the regulator only unless JP1 is bridged. The assembly instructions now
flash with power connected and describe the LED check and JP1.

Co-Authored-By: Claude Opus 5 <noreply@anthropic.com>
Parts:
- JP1: footprint Jumper:SolderJumper-2_P1.3mm_Bridged_RoundedPad1.0x1.5mm -> Jumper:SolderJumper-2_P1.3mm_Open_RoundedPad1.0x1.5mm
Changed lines of the file:
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@@
 		)
 	)
-	(footprint "Jumper:SolderJumper-2_P1.3mm_Bridged_RoundedPad1.0x1.5mm"
+	(footprint "Jumper:SolderJumper-2_P1.3mm_Open_RoundedPad1.0x1.5mm"
 		(layer "F.Cu")
 		(at 141.5 100.2 -90)
-		(descr "SMD Solder Jumper, 1x1.5mm, rounded Pads, 0.3mm gap, bridged with 1 copper strip")
-		(tags "net tie solder jumper bridged")
+		(descr "SMD Solder Jumper, 1x1.5mm, rounded Pads, 0.3mm gap, open")
+		(tags "solder jumper open")
 		(property "Reference" "JP1"
 			(at 0 -1.8 90)
@@
 			)
 		)
-		(property "Description" "Solder Jumper, 2-pole, closed/bridged"
+		(property "Description" "Solder Jumper, 2-pole, open"
 			(at 0 0 270)
 			(unlocked yes)
@@
 			)
 		)
-		(property ki_fp_filters "SolderJumper*Bridged*")
+		(property ki_fp_filters "SolderJumper*Open*")
 		(sheetname "/Power Supply/")
 		(sheetfile "power_supply.kicad_sch")
 		(zone_connect 1)
 		(attr exclude_from_pos_files exclude_from_bom allow_soldermask_bridges)
-		(net_tie_pad_groups "1, 2")
 		(duplicate_pad_numbers_are_jumpers no)
-		(fp_poly
-			(pts
-				(xy 0.25 -0.3) (xy -0.25 -0.3) (xy -0.25 0.3) (xy 0.25 0.3)
-			)
-			(stroke
-				(width 0)
-				(type solid)
-			)
-			(fill yes)
-			(layer "F.Cu")
-		)
 		(fp_rect
 			(start -0.15 -0.75)
