File: pcb/controller/src/motor_driver.kicad_sch (KiCad schematic)
At the start: 11 parts, among them J1 Motor, U3 PDRV8311HRRWR

Commit message: Add manufacturer, MPN and LCSC part numbers to all boards
Part numbers taken from the matched JLCPCB order BOMs. Also mark the RM2
module (U6) and microSD socket (J8) as DNP, exclude test points from the
BOM, use KT-0805B for D7, 100n 50V for C42 as built, and set ENIG as the
surface finish.

Co-Authored-By: Claude Opus 5 <noreply@anthropic.com>
Parts:
- C1: JLCPCB Part # C28241 -> (none); LCSC (none) -> C440198; MPN (none) -> GRM21BR61H106KE43L; Manufacturer (none) -> Murata
- C3: LCSC (none) -> C19702; MPN (none) -> CL10A106KP8NNNC; Manufacturer (none) -> Samsung Electro-Mechanics
- C4, C6: LCSC (none) -> C307331; MPN (none) -> CL05B104KB54PNC; Manufacturer (none) -> Samsung Electro-Mechanics
- C8, C9: LCSC (none) -> C1525; MPN (none) -> CL05B104KO5NNNC; Manufacturer (none) -> Samsung Electro-Mechanics
- D5: LCSC (none) -> C84256; MPN (none) -> NCD0805R1; Manufacturer (none) -> NATIONSTAR
- J1: LCSC (none) -> C293630; MPN (none) -> 532610371; Manufacturer (none) -> Molex
- R34: LCSC (none) -> C11702; MPN (none) -> 0402WGF1001TCE; Manufacturer (none) -> UNI-ROYAL
- R5: LCSC (none) -> C25792; MPN (none) -> 0402WGF4702TCE; Manufacturer (none) -> UNI-ROYAL
- U3: LCSC (none) -> C5218862; MPN (none) -> DRV8311HRRWR; Manufacturer (none) -> Texas Instruments
