File: pcb/controller/src/usb_hub.kicad_sch (KiCad schematic)
At the start: 24 parts, among them IC1 USB2422-I_MJ, J3 USB_C_Receptacle_USB2.0_14P, U5 USBLC6-2P6, Y2 7M-24.000MAAJ-T

Commit message: Add manufacturer, MPN and LCSC part numbers to all boards
Part numbers taken from the matched JLCPCB order BOMs. Also mark the RM2
module (U6) and microSD socket (J8) as DNP, exclude test points from the
BOM, use KT-0805B for D7, 100n 50V for C42 as built, and set ENIG as the
surface finish.

Co-Authored-By: Claude Opus 5 <noreply@anthropic.com>
Parts:
- C22, C24: LCSC (none) -> C52923; MPN (none) -> CL05A105KA5NQNC; Manufacturer (none) -> Samsung Electro-Mechanics
- C23, C25, C26: LCSC (none) -> C1525; MPN (none) -> CL05B104KO5NNNC; Manufacturer (none) -> Samsung Electro-Mechanics
- C39, C40: LCSC (none) -> C1549; MPN (none) -> 0402CG180J500NT; Manufacturer (none) -> Fenghua
- C42: value 100n 250V -> 100n 50V; LCSC (none) -> C77020; MPN (none) -> GRM155R71H104KE14D; Manufacturer (none) -> Murata
- D4: LCSC (none) -> C2296; MPN (none) -> KT-0805Y; Manufacturer (none) -> Hubei KENTO Elec
- IC1: LCSC (none) -> C220747; MANUFACTURER_NAME Microchip -> (none); MANUFACTURER_PART_NUMBER USB2422-I/MJ -> (none); MF Microchip -> (none); MP USB2422-I/MJ -> (none); MPN (none) -> USB2422-I/MJ; Manufacturer (none) -> Microchip
- J3: LCSC (none) -> C3025063; MPN (none) -> USB4105-GF-A-060; Manufacturer (none) -> Global Connector Technology
- R11: LCSC (none) -> C163474; MPN (none) -> RC0402FR-07270RL; Manufacturer (none) -> Yageo
- R19, R20: LCSC (none) -> C25741; MPN (none) -> 0402WGF1003TCE; Manufacturer (none) -> UNI-ROYAL
- R21: LCSC (none) -> C25752; MPN (none) -> 0402WGF1202TCE; Manufacturer (none) -> UNI-ROYAL
- R22, R23, R24, R26: LCSC (none) -> C25792; MPN (none) -> 0402WGF4702TCE; Manufacturer (none) -> UNI-ROYAL
- R25, R27: LCSC (none) -> C25768; MPN (none) -> 0402WGF2202TCE; Manufacturer (none) -> UNI-ROYAL
- R28: LCSC (none) -> C25104; MPN (none) -> 0402WGF3300TCE; Manufacturer (none) -> UNI-ROYAL
- U5: LCSC (none) -> C2827693; MPN (none) -> USBLC6-2P6; Manufacturer (none) -> TECH PUBLIC
- Y2: LCSC (none) -> C2450233; MANUFACTURER ABRACON -> (none); MF ABRACON -> (none); MP ABM8-272-T3 -> (none); MPN (none) -> 7M-24.000MAAJ-T; Manufacturer (none) -> TXC
