File: pcb/controller/src/OWL - Rotor v2.kicad_sch (KiCad schematic)
At the start: 11 parts, among them J4 Slip Ring

Commit message: Add manufacturer, MPN and LCSC part numbers to all boards
Part numbers taken from the matched JLCPCB order BOMs. Also mark the RM2
module (U6) and microSD socket (J8) as DNP, exclude test points from the
BOM, use KT-0805B for D7, 100n 50V for C42 as built, and set ENIG as the
surface finish.

Co-Authored-By: Claude Opus 5 <noreply@anthropic.com>
Parts:
- D2, D8, D9: LCSC (none) -> C2297; MPN (none) -> KT-0805G; Manufacturer (none) -> Hubei KENTO Elec
- J4: LCSC (none) -> C265376; MPN (none) -> BM06B-PASS-TFT(LF)(SN); Manufacturer (none) -> JST
- R3: LCSC (none) -> C25123; MPN (none) -> 0402WGF5100TCE; Manufacturer (none) -> UNI-ROYAL
- R39: LCSC (none) -> C25900; MPN (none) -> 0402WGF4701TCE; Manufacturer (none) -> UNI-ROYAL
- R40: LCSC (none) -> C25082; MPN (none) -> 0402WGF1500TCE; Manufacturer (none) -> UNI-ROYAL
- TP6, TP7, TP8, TP9: now left out of the parts list
Changed lines of the file:
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@@
+			)
+		)
+		(property "Manufacturer" "UNI-ROYAL"
+			(at 227.33 101.6 0)
+			(hide yes)
+			(show_name no)
+			(do_not_autoplace no)
+			(effects
+				(font
+					(size 1.27 1.27)
+				)
+			)
+		)
+		(property "MPN" "0402WGF5100TCE"
+			(at 227.33 101.6 0)
+			(hide yes)
+			(show_name no)
+			(do_not_autoplace no)
+			(effects
+				(font
+					(size 1.27 1.27)
+				)
+			)
+		)
+		(property "LCSC" "C25123"
+			(at 227.33 101.6 0)
+			(hide yes)
+			(show_name no)
+			(do_not_autoplace no)
+			(effects
+				(font
+					(size 1.27 1.27)
+				)
 			)
 		)
@@
 			)
 		)
+		(property "Manufacturer" "Hubei KENTO Elec"
+			(at 262.89 91.44 0)
+			(hide yes)
+			(show_name no)
+			(do_not_autoplace no)
+			(effects
+				(font
+					(size 1.27 1.27)
+				)
+			)
+		)
+		(property "MPN" "KT-0805G"
+			(at 262.89 91.44 0)
+			(hide yes)
+			(show_name no)
+			(do_not_autoplace no)
+			(effects
+				(font
+					(size 1.27 1.27)
+				)
+			)
+		)
+		(property "LCSC" "C2297"
+			(at 262.89 91.44 0)
+			(hide yes)
+			(show_name no)
+			(do_not_autoplace no)
+			(effects
+				(font
+					(size 1.27 1.27)
+				)
+			)
+		)
 		(pin "1"
 		)
@@
 			)
 		)
+		(property "Manufacturer" "UNI-ROYAL"
+			(at 245.11 101.6 0)
+			(hide yes)
+			(show_name no)
+			(do_not_autoplace no)
+			(effects
+				(font
+					(size 1.27 1.27)
+				)
+			)
+		)
+		(property "MPN" "0402WGF4701TCE"
+			(at 245.11 101.6 0)
+			(hide yes)
+			(show_name no)
+			(do_not_autoplace no)
+			(effects
+				(font
+					(size 1.27 1.27)
+				)
+			)
+		)
+		(property "LCSC" "C25900"
+			(at 245.11 101.6 0)
+			(hide yes)
+			(show_name no)
+			(do_not_autoplace no)
+			(effects
+				(font
+					(size 1.27 1.27)
+				)
+			)
+		)
 		(pin "1"
 		)
@@
 		(body_style 1)
 		(exclude_from_sim no)
-		(in_bom yes)
+		(in_bom no)
 		(on_board yes)
 		(in_pos_files yes)
@@
 			)
 		)
+		(property "Manufacturer" "UNI-ROYAL"
+			(at 262.89 101.6 0)
+			(hide yes)
+			(show_name no)
+			(do_not_autoplace no)
+			(effects
+				(font
+					(size 1.27 1.27)
+				)
+			)
+		)
+		(property "MPN" "0402WGF1500TCE"
+			(at 262.89 101.6 0)
+			(hide yes)
+			(show_name no)
+			(do_not_autoplace no)
+			(effects
+				(font
+					(size 1.27 1.27)
+				)
+			)
+		)
+		(property "LCSC" "C25082"
+			(at 262.89 101.6 0)
+			(hide yes)
+			(show_name no)
+			(do_not_autoplace no)
+			(effects
+				(font
+					(size 1.27 1.27)
+				)
+			)
+		)
 		(pin "1"
 		)
@@
 		(body_style 1)
 		(exclude_from_sim no)
-		(in_bom yes)
+		(in_bom no)
 		(on_board yes)
 		(in_pos_files yes)
@@
 		(body_style 1)
 		(exclude_from_sim no)
-		(in_bom yes)
+		(in_bom no)
 		(on_board yes)
 		(in_pos_files yes)
@@
 			)
 		)
+		(property "Manufacturer" "Hubei KENTO Elec"
+			(at 227.33 91.44 0)
+			(hide yes)
+			(show_name no)
+			(do_not_autoplace no)
+			(effects
+				(font
+					(size 1.27 1.27)
+				)
+			)
+		)
+		(property "MPN" "KT-0805G"
+			(at 227.33 91.44 0)
+			(hide yes)
+			(show_name no)
+			(do_not_autoplace no)
+			(effects
+				(font
+					(size 1.27 1.27)
+				)
+			)
+		)
+		(property "LCSC" "C2297"
+			(at 227.33 91.44 0)
+			(hide yes)
+			(show_name no)
+			(do_not_autoplace no)
+			(effects
+				(font
+					(size 1.27 1.27)
+				)
+			)
+		)
 		(pin "1"
 		)
@@
 		(body_style 1)
 		(exclude_from_sim no)
-		(in_bom yes)
+		(in_bom no)
 		(on_board yes)
 		(in_pos_files yes)
@@
 			)
 		)
+		(property "Manufacturer" "JST"
+			(at 227.33 50.8 0)
+			(hide yes)
+			(show_name no)
+			(do_not_autoplace no)
+			(effects
+				(font
+					(size 1.27 1.27)
+				)
+			)
+		)
+		(property "MPN" "BM06B-PASS-TFT(LF)(SN)"
+			(at 227.33 50.8 0)
+			(hide yes)
+			(show_name no)
+			(do_not_autoplace no)
+			(effects
+				(font
+					(size 1.27 1.27)
+				)
+			)
+		)
+		(property "LCSC" "C265376"
+			(at 227.33 50.8 0)
+			(hide yes)
+			(show_name no)
+			(do_not_autoplace no)
+			(effects
+				(font
+					(size 1.27 1.27)
+				)
+			)
+		)
 		(pin "6"
 		)
@@
 			(at 245.11 91.44 0)
 			(hide yes)
+			(show_name no)
+			(do_not_autoplace no)
+			(effects
+				(font
+					(size 1.27 1.27)
+				)
+			)
+		)
+		(property "Manufacturer" "Hubei KENTO Elec"
+			(at 245.11 91.44 0)
+			(hide yes)
+			(show_name no)
+			(do_not_autoplace no)
+			(effects
+				(font
+					(size 1.27 1.27)
+				)
+			)
+		)
+		(property "MPN" "KT-0805G"
+			(at 245.11 91.44 0)
+			(hide yes)
+			(show_name no)
+			(do_not_autoplace no)
+			(effects
+				(font
+					(size 1.27 1.27)
+				)
+			)
+		)
+		(property "LCSC" "C2297"
+			(at 245.11 91.44 0)
+			(hide yes)

Commit message: Lower the current of the green 5V and 3.3V LEDs
R3 510 -> 1.43k and R40 150 -> 360, about 1.5 mA like the VM LED
instead of 3-4 mA. Both values are already in the BOM.

Co-Authored-By: Claude Opus 5 <noreply@anthropic.com>
Parts:
- R3: value 510 -> 1.43k; LCSC C25123 -> C163483; MPN 0402WGF5100TCE -> RC0402FR-071K43L; Manufacturer UNI-ROYAL -> Yageo
- R40: value 150 -> 360; LCSC C25082 -> C2930003; MPN 0402WGF1500TCE -> FRC0402F3600TS; Manufacturer UNI-ROYAL -> FOJAN
Changed lines of the file:
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@@
 			)
 		)
-		(property "Value" "510"
+		(property "Value" "1.43k"
 			(at 229.87 102.8699 0)
 			(show_name no)
@@
 			)
 		)
-		(property "Manufacturer" "UNI-ROYAL"
+		(property "Manufacturer" "Yageo"
 			(at 227.33 101.6 0)
 			(hide yes)
@@
 			)
 		)
-		(property "MPN" "0402WGF5100TCE"
+		(property "MPN" "RC0402FR-071K43L"
 			(at 227.33 101.6 0)
 			(hide yes)
@@
 			)
 		)
-		(property "LCSC" "C25123"
+		(property "LCSC" "C163483"
 			(at 227.33 101.6 0)
 			(hide yes)
@@
 			)
 		)
-		(property "Value" "150"
+		(property "Value" "360"
 			(at 265.43 102.8699 0)
 			(show_name no)
@@
 			)
 		)
-		(property "Manufacturer" "UNI-ROYAL"
+		(property "Manufacturer" "FOJAN"
 			(at 262.89 101.6 0)
 			(hide yes)
@@
 			)
 		)
-		(property "MPN" "0402WGF1500TCE"
+		(property "MPN" "FRC0402F3600TS"
 			(at 262.89 101.6 0)
 			(hide yes)
@@
 			)
 		)
-		(property "LCSC" "C25082"
+		(property "LCSC" "C2930003"
 			(at 262.89 101.6 0)
 			(hide yes)
