File: pcb/controller/src/power_supply.kicad_sch (KiCad schematic)
At the start: 25 parts, among them U1 AP2112K-3.3, U2 LM66200DRLR

Commit message: Add manufacturer, MPN and LCSC part numbers to all boards
Part numbers taken from the matched JLCPCB order BOMs. Also mark the RM2
module (U6) and microSD socket (J8) as DNP, exclude test points from the
BOM, use KT-0805B for D7, 100n 50V for C42 as built, and set ENIG as the
surface finish.

Co-Authored-By: Claude Opus 5 <noreply@anthropic.com>
Parts:
- C10, C11: LCSC (none) -> C19702; MPN (none) -> CL10A106KP8NNNC; Manufacturer (none) -> Samsung Electro-Mechanics
- C31, C32, C33: LCSC (none) -> C440198; MPN (none) -> GRM21BR61H106KE43L; Manufacturer (none) -> Murata
- C34: LCSC (none) -> C307331; MPN (none) -> CL05B104KB54PNC; Manufacturer (none) -> Samsung Electro-Mechanics
- C35, C36, C37: LCSC (none) -> C60077; MPN (none) -> 0603X226M100NT; Manufacturer (none) -> Fenghua
- C38: LCSC (none) -> C1525; MPN (none) -> CL05B104KO5NNNC; Manufacturer (none) -> Samsung Electro-Mechanics
- D6: LCSC (none) -> C84256; MPN (none) -> NCD0805R1; Manufacturer (none) -> NATIONSTAR
- PS1: LCSC (none) -> C47122151; MANUFACTURER Texas Instruments -> (none); MF Texas Instruments -> (none); MP TPSM84338RCJR -> (none); MPN (none) -> TPSM84338RCJR; Manufacturer (none) -> Texas Instruments
- R29: LCSC (none) -> C138065; MPN (none) -> RC0402FR-07110KL; Manufacturer (none) -> Yageo
- R30: LCSC (none) -> C25756; MPN (none) -> 0402WGF1502TCE; Manufacturer (none) -> UNI-ROYAL
- R31: LCSC (none) -> C17168; MPN (none) -> 0402WGF0000TCE; Manufacturer (none) -> UNI-ROYAL
- R32: LCSC (none) -> C25762; MPN (none) -> 0402WGF1802TCE; Manufacturer (none) -> UNI-ROYAL
- R36: LCSC (none) -> C11702; MPN (none) -> 0402WGF1001TCE; Manufacturer (none) -> UNI-ROYAL
- TP1, TP2, TP3, TP4: now left out of the parts list
- U1: MPN (none) -> AP2112K-3.3TRG1; Manufacturer (none) -> TECH PUBLIC
- U2: LCSC (none) -> C3235556; MPN (none) -> LM66200DRLR; Manufacturer (none) -> Texas Instruments

Commit message: Ship the controller VBUS jumper JP1 open
With both USB VBUS and the regulator connected, the LM66200 keeps
switching between the two nearly equal inputs and the 5V rail gets
noisy. JP1 is now an open solder jumper, so the controller runs from
the regulator only unless JP1 is bridged. The assembly instructions now
flash with power connected and describe the LED check and JP1.

Co-Authored-By: Claude Opus 5 <noreply@anthropic.com>
Parts:
- JP1: footprint Jumper:SolderJumper-2_P1.3mm_Bridged_RoundedPad1.0x1.5mm -> Jumper:SolderJumper-2_P1.3mm_Open_RoundedPad1.0x1.5mm; symbol Jumper:SolderJumper_2_Bridged -> Jumper:SolderJumper_2_Open
Changed lines of the file:
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@@
 	)
 	(symbol
-		(lib_id "Jumper:SolderJumper_2_Bridged")
+		(lib_id "Jumper:SolderJumper_2_Open")
 		(at 182.88 129.54 0)
 		(mirror y)
@@
 			)
 		)
-		(property "Footprint" "Jumper:SolderJumper-2_P1.3mm_Bridged_RoundedPad1.0x1.5mm"
+		(property "Footprint" "Jumper:SolderJumper-2_P1.3mm_Open_RoundedPad1.0x1.5mm"
 			(at 182.88 129.54 0)
 			(hide yes)
@@
 			)
 		)
-		(property "Description" "Solder Jumper, 2-pole, closed/bridged"
+		(property "Description" "Solder Jumper, 2-pole, open"
 			(at 182.88 129.54 0)
 			(hide yes)
