File: pcb/controller/src/rp2354b.kicad_sch (KiCad schematic)
At the start: 43 parts, among them J5 781715006, J6 SM03B-SRSS-TB, J8 Micro_SD_Card, J9 SM04B-SRSS-TB_LF__SN_, SW1 BOOTSEL, SW2 RESET, SW3 USER, U4 RP2354B, Y1 ABM8-272-T3

Commit message: Add manufacturer, MPN and LCSC part numbers to all boards
Part numbers taken from the matched JLCPCB order BOMs. Also mark the RM2
module (U6) and microSD socket (J8) as DNP, exclude test points from the
BOM, use KT-0805B for D7, 100n 50V for C42 as built, and set ENIG as the
surface finish.

Co-Authored-By: Claude Opus 5 <noreply@anthropic.com>
Parts:
- C12, C13, C15, C16, C17, C18, C21, C27, C28, C29, C30, C43: LCSC (none) -> C1525; MPN (none) -> CL05B104KO5NNNC; Manufacturer (none) -> Samsung Electro-Mechanics
- C14, C2, C5, C7: LCSC (none) -> C23733; MPN (none) -> CL05A475MP5NRNC; Manufacturer (none) -> Samsung Electro-Mechanics
- C19, C20: LCSC (none) -> C1548; MPN (none) -> 0402CG150J500NT; Manufacturer (none) -> Fenghua
- C44: LCSC (none) -> C19702; MPN (none) -> CL10A106KP8NNNC; Manufacturer (none) -> Samsung Electro-Mechanics
- D7: LCSC (none) -> C2293; MPN (none) -> KT-0805B; Manufacturer (none) -> Hubei KENTO Elec
- J5: LCSC (none) -> C107412; MANUFACTURER_PART_NUMBER 781715006 -> (none); MF Molex -> (none); MFR_NAME Molex Connector Corporation -> (none); MP 781715006 -> (none); MPN (none) -> 781715006; Manufacturer (none) -> Molex
- J6: LCSC (none) -> C160403; MPN (none) -> SM03B-SRSS-TB(LF)(SN); Manufacturer (none) -> JST
- J8: now not fitted
- J9: MANUFACTURER JST -> (none); MF JST Sales -> (none); MP SM04B-SRSS-TB (LF)(SN) -> (none); MPN (none) -> SM04B-SRSS-TB(LF)(SN); Manufacturer (none) -> JST
- L1: LCSC (none) -> C42411119; MPN (none) -> AOTA-B201610S3R3-101-T; Manufacturer (none) -> Abracon
- R13: LCSC (none) -> C25105; MPN (none) -> 0402WGF330JTCE; Manufacturer (none) -> UNI-ROYAL
- R14, R15, R18, R41: LCSC (none) -> C11702; MPN (none) -> 0402WGF1001TCE; Manufacturer (none) -> UNI-ROYAL
- R16, R17: LCSC (none) -> C138021; MPN (none) -> RC0402FR-0727RL; Manufacturer (none) -> Yageo
- R38: LCSC (none) -> C2930003; MPN (none) -> FRC0402F3600TS; Manufacturer (none) -> FOJAN
- R4: LCSC (none) -> C25744; MPN (none) -> 0402WGF1002TCE; Manufacturer (none) -> UNI-ROYAL
- R6: LCSC (none) -> C163483; MPN (none) -> RC0402FR-071K43L; Manufacturer (none) -> Yageo
- SW1, SW2, SW3: LCSC (none) -> C843684; MPN (none) -> GT-TC032A-H015-L1; Manufacturer (none) -> G-Switch
- TP10, TP12, TP5: now left out of the parts list
- U4: LCSC (none) -> C39843328; MPN (none) -> RP2354B; Manufacturer (none) -> Raspberry Pi
- Y1: LCSC (none) -> C20625731; MANUFACTURER ABRACON -> (none); MF ABRACON -> (none); MP ABM8-272-T3 -> (none); MPN (none) -> ABM8-272-T3; Manufacturer (none) -> Abracon

Commit message: Assemble the controller on the top side only
Mark C43, C44 (bulk decoupling for the microSD socket and RM2 module)
and R1, R2 (RM2 only) as DNP like J8 and U6, so the controller has no
assembled bottom-side parts. They can still be hand-soldered.

Co-Authored-By: Claude Opus 5 <noreply@anthropic.com>
Parts:
- C43, C44: now not fitted
Changed lines of the file:
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@@
 		(on_board yes)
 		(in_pos_files yes)
-		(dnp no)
+		(dnp yes)
 		(property "Reference" "C44"
 			(at 202.946 90.678 0)
@@
 		(on_board yes)
 		(in_pos_files yes)
-		(dnp no)
+		(dnp yes)
 		(property "Reference" "C43"
 			(at 188.976 90.424 0)
