File: pcb/sensor/ma600a/src/Sensor - MA600A.kicad_sch (KiCad schematic)
At the start: 6 parts, among them J1 781715006, U2 MA600A

Commit message: Add manufacturer, MPN and LCSC part numbers to all boards
Part numbers taken from the matched JLCPCB order BOMs. Also mark the RM2
module (U6) and microSD socket (J8) as DNP, exclude test points from the
BOM, use KT-0805B for D7, 100n 50V for C42 as built, and set ENIG as the
surface finish.

Co-Authored-By: Claude Opus 5 <noreply@anthropic.com>
Parts:
- C1: LCSC (none) -> C14663; MPN (none) -> CC0603KRX7R9BB104; Manufacturer (none) -> Yageo
- C2: LCSC (none) -> C15849; MPN (none) -> CL10A105KB8NNNC; Manufacturer (none) -> Samsung Electro-Mechanics
- J1: LCSC (none) -> C107412; MANUFACTURER_PART_NUMBER 781715006 -> (none); MF Molex -> (none); MFR_NAME Molex Connector Corporation -> (none); MP 781715006 -> (none); MPN (none) -> 781715006; Manufacturer (none) -> Molex
- TP1, TP2: now left out of the parts list
- U2: LCSC (none) -> C49240579; MPN (none) -> MA600AGQE-0000-Z; Manufacturer (none) -> Monolithic Power Systems
Changed lines of the file:
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@@
 			)
 		)
-		(property "MF" "Molex"
+		(property "Description_1" "Conn Wire to Board HDR 6 POS 1.2mm Solder ST Top Entry SMD Pico-EZmate™ T/R"
 			(at 229.87 97.79 0)
 			(effects
@@
 			)
 		)
-		(property "Description_1" "Conn Wire to Board HDR 6 POS 1.2mm Solder ST Top Entry SMD Pico-EZmate™ T/R"
+		(property "Package" "None"
 			(at 229.87 97.79 0)
 			(effects
@@
 			)
 		)
-		(property "Package" "None"
+		(property "Price" "None"
 			(at 229.87 97.79 0)
 			(effects
@@
 			)
 		)
-		(property "Price" "None"
+		(property "Check_prices" "https://www.snapeda.com/parts/781715006/Molex/view-part/?ref=eda"
 			(at 229.87 97.79 0)
 			(effects
@@
 			)
 		)
-		(property "Check_prices" "https://www.snapeda.com/parts/781715006/Molex/view-part/?ref=eda"
+		(property "Availability" "In Stock"
 			(at 229.87 97.79 0)
 			(effects
@@
 			)
 		)
-		(property "Availability" "In Stock"
+		(property "SnapEDA_Link" "https://www.snapeda.com/parts/781715006/Molex/view-part/?ref=snap"
 			(at 229.87 97.79 0)
 			(effects
@@
 			)
 		)
-		(property "SnapEDA_Link" "https://www.snapeda.com/parts/781715006/Molex/view-part/?ref=snap"
-			(at 229.87 97.79 0)
-			(effects
-				(font
-					(size 1.27 1.27)
-				)
-				(justify bottom)
-				(hide yes)
-			)
-		)
-		(property "MP" "781715006"
-			(at 229.87 97.79 0)
-			(effects
-				(font
-					(size 1.27 1.27)
-				)
-				(justify bottom)
-				(hide yes)
-			)
-		)
-		(property "MFR_NAME" "Molex Connector Corporation"
-			(at 229.87 97.79 0)
-			(effects
-				(font
-					(size 1.27 1.27)
-				)
-				(justify bottom)
-				(hide yes)
-			)
-		)
-		(property "MANUFACTURER_PART_NUMBER" "781715006"
-			(at 229.87 97.79 0)
-			(effects
-				(font
-					(size 1.27 1.27)
-				)
-				(justify bottom)
-				(hide yes)
+		(property "Manufacturer" "Molex"
+			(at 229.87 97.79 0)
+			(hide yes)
+			(show_name no)
+			(do_not_autoplace no)
+			(effects
+				(font
+					(size 1.27 1.27)
+				)
+			)
+		)
+		(property "MPN" "781715006"
+			(at 229.87 97.79 0)
+			(hide yes)
+			(show_name no)
+			(do_not_autoplace no)
+			(effects
+				(font
+					(size 1.27 1.27)
+				)
+			)
+		)
+		(property "LCSC" "C107412"
+			(at 229.87 97.79 0)
+			(hide yes)
+			(show_name no)
+			(do_not_autoplace no)
+			(effects
+				(font
+					(size 1.27 1.27)
+				)
 			)
 		)
@@
 		(unit 1)
 		(exclude_from_sim no)
-		(in_bom yes)
+		(in_bom no)
 		(on_board yes)
 		(dnp no)
@@
 			)
 		)
+		(property "Manufacturer" "Samsung Electro-Mechanics"
+			(at 168.91 92.71 0)
+			(hide yes)
+			(show_name no)
+			(do_not_autoplace no)
+			(effects
+				(font
+					(size 1.27 1.27)
+				)
+			)
+		)
+		(property "MPN" "CL10A105KB8NNNC"
+			(at 168.91 92.71 0)
+			(hide yes)
+			(show_name no)
+			(do_not_autoplace no)
+			(effects
+				(font
+					(size 1.27 1.27)
+				)
+			)
+		)
+		(property "LCSC" "C15849"
+			(at 168.91 92.71 0)
+			(hide yes)
+			(show_name no)
+			(do_not_autoplace no)
+			(effects
+				(font
+					(size 1.27 1.27)
+				)
+			)
+		)
 		(pin "1"
 		)
@@
 			)
 		)
+		(property "Manufacturer" "Yageo"
+			(at 181.61 92.71 0)
+			(hide yes)
+			(show_name no)
+			(do_not_autoplace no)
+			(effects
+				(font
+					(size 1.27 1.27)
+				)
+			)
+		)
+		(property "MPN" "CC0603KRX7R9BB104"
+			(at 181.61 92.71 0)
+			(hide yes)
+			(show_name no)
+			(do_not_autoplace no)
+			(effects
+				(font
+					(size 1.27 1.27)
+				)
+			)
+		)
+		(property "LCSC" "C14663"
+			(at 181.61 92.71 0)
+			(hide yes)
+			(show_name no)
+			(do_not_autoplace no)
+			(effects
+				(font
+					(size 1.27 1.27)
+				)
+			)
+		)
 		(pin "1"
 		)
@@
 			)
 		)
+		(property "Manufacturer" "Monolithic Power Systems"
+			(at 132.08 91.44 0)
+			(hide yes)
+			(show_name no)
+			(do_not_autoplace no)
+			(effects
+				(font
+					(size 1.27 1.27)
+				)
+			)
+		)
+		(property "MPN" "MA600AGQE-0000-Z"
+			(at 132.08 91.44 0)
+			(hide yes)
+			(show_name no)
+			(do_not_autoplace no)
+			(effects
+				(font
+					(size 1.27 1.27)
+				)
+			)
+		)
+		(property "LCSC" "C49240579"
+			(at 132.08 91.44 0)
+			(hide yes)
+			(show_name no)
+			(do_not_autoplace no)
+			(effects
+				(font
+					(size 1.27 1.27)
+				)
+			)
+		)
 		(pin "5"
 		)
@@
 		(unit 1)
 		(exclude_from_sim no)
-		(in_bom yes)
+		(in_bom no)
 		(on_board yes)
 		(dnp no)
