File: pcb/stator/src/Stator.kicad_sch (KiCad schematic)
At the start: 22 parts, among them J1 DATA, J2 SLIP RING, J3 POWER, U2 CH224K

Commit message: Add manufacturer, MPN and LCSC part numbers to all boards
Part numbers taken from the matched JLCPCB order BOMs. Also mark the RM2
module (U6) and microSD socket (J8) as DNP, exclude test points from the
BOM, use KT-0805B for D7, 100n 50V for C42 as built, and set ENIG as the
surface finish.

Co-Authored-By: Claude Opus 5 <noreply@anthropic.com>
Parts:
- C1, C4: LCSC (none) -> C1581; MPN (none) -> 0402F104M500NT; Manufacturer (none) -> Fenghua
- C3: LCSC (none) -> C52923; MPN (none) -> CL05A105KA5NQNC; Manufacturer (none) -> Samsung Electro-Mechanics
- J1, J3: LCSC (none) -> C5143397; MPN (none) -> USB4110-GF-A; Manufacturer (none) -> Global Connector Technology
- J2: MPN (none) -> BM06B-PASS-TFT(LF)(SN); Manufacturer (none) -> JST
- R1, R6: LCSC (none) -> C25104; MPN (none) -> 0402WGF3300TCE; Manufacturer (none) -> UNI-ROYAL
- R2, R3: LCSC (none) -> C25905; MPN (none) -> 0402WGF5101TCE; Manufacturer (none) -> UNI-ROYAL
- R4, R7, R8, R9: LCSC (none) -> C25744; MPN (none) -> 0402WGF1002TCE; Manufacturer (none) -> UNI-ROYAL
- R5: LCSC (none) -> C560481; MPN (none) -> AS05W2J0102T5E; Manufacturer (none) -> UNI-ROYAL
- TP1, TP2, TP3: now left out of the parts list
- U2: MPN (none) -> CH224K; Manufacturer (none) -> WCH
