File: pcb/stator/src/Stator.kicad_pcb (KiCad board)
At the start: 2 copper layers, 44 x 44 mm, 22 parts, among them J1 DATA, J2 SLIP RING, J3 POWER, U2 CH224K

Commit message: Route the second D+/D- pads of the stator data USB-C port
J1 B6 and B7 were not connected, so the port only worked in one
orientation.

Co-Authored-By: Claude Opus 5 <noreply@anthropic.com>
Routing:
- net /USB_D-: track 35.4 -> 37.4 mm
- net /USB_D+: track 35.3 -> 37.0 mm, vias 0 -> 2
